Commit message: mr robot urdf

File: fcl_coll/urdf/robot_arm.urdf (robot description, URDF)
Before this commit: robot simple_2dof_arm, 3 links, 2 joints
Links:
- removed link link1
- removed link link2
- added link left_wheel, mass 0.3; collision cylinder length=0.02 radius=0.05; visual cylinder length=0.02 radius=0.05
- added link right_wheel, mass 0.3; collision cylinder length=0.02 radius=0.05; visual cylinder length=0.02 radius=0.05
- link base_link: mass None -> 5.0; geometry collision box size=0.4 0.3 0.1; visual box size=0.4 0.3 0.1
Joints:
- removed joint joint1
- removed joint joint2
- added joint left_wheel_joint: type continuous, parent base_link, child left_wheel, origin xyz=0 0.15 -0.06 rpy=0 0 0, axis 0 1 0
- added joint right_wheel_joint: type continuous, parent base_link, child right_wheel, origin xyz=0 -0.15 -0.06 rpy=0 0 0, axis 0 1 0

File: fcl_coll/urdf2/mr_robot.xacro (robot description, xacro)
@@ -1,7 +1,7 @@
 <?xml version="1.0" ?>
 <robot name="mr_robot" xmlns:xacro="http://www.ros.org/wiki/xacro">
-<xacro:include filename="$(find mr_robot_description)/urdf/materials.xacro" />
-<xacro:include filename="$(find mr_robot_description)/urdf/mr_robot.trans" />
-<xacro:include filename="$(find mr_robot_description)/urdf/mr_robot.gazebo" />
+<xacro:include filename="$(find fcl_coll)/urdf/materials.xacro" />
+<xacro:include filename="$(find fcl_coll)/urdf/mr_robot.trans" />
+<xacro:include filename="$(find fcl_coll)/urdf/mr_robot.gazebo" />
 <!-- BASE FOOTPRINT LINK -->
 <link name="base_footprint">
@@ -21,5 +21,5 @@
     <origin xyz="0 0 0" rpy="0 0 0"/>
     <geometry>
-      <mesh filename="file://$(find mr_robot_description)/meshes/base_link.stl" scale="0.001 0.001 0.001"/>
+     <box size="0.5 0.3 0.1"/>
     </geometry>
     <material name="silver"/>
@@ -28,5 +28,5 @@
     <origin xyz="0 0 0" rpy="0 0 0"/>
     <geometry>
-      <mesh filename="file://$(find mr_robot_description)/meshes/base_link.stl" scale="0.001 0.001 0.001"/>
+      <box size="0.5 0.3 0.1"/>
     </geometry>
   </collision>
@@ -39,14 +39,14 @@
   </inertial>
   <visual>
-    <origin xyz="-0.0 0.172825 0.0556" rpy="0 0 0"/>
+    <origin xyz="-0.0 0.172825 0.0556" rpy="1.5708 0 0"/>
     <geometry>
-      <mesh filename="file://$(find mr_robot_description)/meshes/right_wheel__1.stl" scale="0.001 0.001 0.001"/>
+      <cylinder radius="0.05" length="0.02"/>
     </geometry>
     <material name="silver"/>
   </visual>
   <collision>
-    <origin xyz="-0.0 0.172825 0.0556" rpy="0 0 0"/>
+    <origin xyz="-0.0 0.172825 0.0556" rpy="1.5708 0 0"/>
     <geometry>
-      <mesh filename="file://$(find mr_robot_description)/meshes/right_wheel__1.stl" scale="0.001 0.001 0.001"/>
+     <cylinder radius="0.05" length="0.02"/>
     </geometry>
   </collision>
@@ -59,14 +59,14 @@
   </inertial>
   <visual>
-    <origin xyz="0.0 -0.181075 0.0556" rpy="0 0 0"/>
+    <origin xyz="0.0 -0.181075 0.0556" rpy="1.5708 0 0"/>
     <geometry>
-      <mesh filename="file://$(find mr_robot_description)/meshes/left_wheel_1.stl" scale="0.001 0.001 0.001"/>
+      <cylinder radius="0.05" length="0.02"/>
     </geometry>
     <material name="silver"/>
   </visual>
   <collision>
-    <origin xyz="0.0 -0.181075 0.0556" rpy="0 0 0"/>
+    <origin xyz="0.0 -0.181075 0.0556" rpy="1.5708 0 0"/>
     <geometry>
-      <mesh filename="file://$(find mr_robot_description)/meshes/left_wheel_1.stl" scale="0.001 0.001 0.001"/>
+      <cylinder radius="0.05" length="0.02"/>
     </geometry>
   </collision>
@@ -81,5 +81,5 @@
     <origin xyz="-0.0 -0.0 -0.0" rpy="0 0 0"/>
     <geometry>
-      <mesh filename="file://$(find mr_robot_description)/meshes/imu_1.stl" scale="0.001 0.001 0.001"/>
+      <cylinder radius="0.05" length="0.02"/>
     </geometry>
     <material name="silver"/>
@@ -88,5 +88,5 @@
     <origin xyz="-0.0 -0.0 -0.0" rpy="0 0 0"/>
     <geometry>
-      <mesh filename="file://$(find mr_robot_description)/meshes/imu_1.stl" scale="0.001 0.001 0.001"/>
+      <cylinder radius="0.05" length="0.02"/>
     </geometry>
   </collision>
@@ -101,5 +101,5 @@
     <origin xyz="-0.087 -0.0 -0.0065" rpy="0 0 0"/>
     <geometry>
-      <mesh filename="file://$(find mr_robot_description)/meshes/gps_1.stl" scale="0.001 0.001 0.001"/>
+      <cylinder radius="0.05" length="0.02"/>
     </geometry>
     <material name="silver"/>
@@ -108,5 +108,5 @@
     <origin xyz="-0.087 -0.0 -0.0065" rpy="0 0 0"/>
     <geometry>
-      <mesh filename="file://$(find mr_robot_description)/meshes/gps_1.stl" scale="0.001 0.001 0.001"/>
+      <cylinder radius="0.05" length="0.02"/>
     </geometry>
   </collision>
@@ -121,5 +121,5 @@
     <origin xyz="-0.2625 -0.0 -0.0085" rpy="0 0 0"/>
     <geometry>
-      <mesh filename="file://$(find mr_robot_description)/meshes/Lidar_1.stl" scale="0.001 0.001 0.001"/>
+      <cylinder radius="0.05" length="0.02"/>
     </geometry>
     <material name="silver"/>
@@ -128,5 +128,5 @@
     <origin xyz="-0.2625 -0.0 -0.0085" rpy="0 0 0"/>
     <geometry>
-      <mesh filename="file://$(find mr_robot_description)/meshes/Lidar_1.stl" scale="0.001 0.001 0.001"/>
+     <cylinder radius="0.05" length="0.02"/>
     </geometry>
   </collision>
