Commit message: meshes parsed

File: fcl_coll/urdf2/mr_robot.xacro (robot description, xacro)
@@ -21,5 +21,5 @@
     <origin xyz="0 0 0" rpy="0 0 0"/>
     <geometry>
-     <box size="0.5 0.3 0.1"/>
+      <mesh filename="package://fcl_coll/meshes/base_link.stl" scale="0.001 0.001 0.001"/>
     </geometry>
     <material name="silver"/>
@@ -28,5 +28,5 @@
     <origin xyz="0 0 0" rpy="0 0 0"/>
     <geometry>
-      <box size="0.5 0.3 0.1"/>
+      <mesh filename="package://fcl_coll/meshes/base_link.stl" scale="0.001 0.001 0.001"/>
     </geometry>
   </collision>
@@ -39,14 +39,14 @@
   </inertial>
   <visual>
-    <origin xyz="-0.0 0.172825 0.0556" rpy="1.5708 0 0"/>
+    <origin xyz="0.0 0.4 0.0" rpy="0 0 0"/>
     <geometry>
-      <cylinder radius="0.05" length="0.02"/>
+      <mesh filename="package://fcl_coll/meshes/right_wheel__1.stl" scale="0.001 0.001 0.001"/>
     </geometry>
     <material name="silver"/>
   </visual>
   <collision>
-    <origin xyz="-0.0 0.172825 0.0556" rpy="1.5708 0 0"/>
+    <origin xyz="0.0 0.4 0.0" rpy="0 0 0"/>
     <geometry>
-     <cylinder radius="0.05" length="0.02"/>
+      <mesh filename="package://fcl_coll/meshes/right_wheel__1.stl" scale="0.001 0.001 0.001"/>
     </geometry>
   </collision>
@@ -59,14 +59,14 @@
   </inertial>
   <visual>
-    <origin xyz="0.0 -0.181075 0.0556" rpy="1.5708 0 0"/>
+    <origin xyz="0.0 -0.4 0.0" rpy="0 0 0"/>
     <geometry>
-      <cylinder radius="0.05" length="0.02"/>
+      <mesh filename="package://fcl_coll/meshes/left_wheel_1.stl" scale="0.001 0.001 0.001"/>
     </geometry>
     <material name="silver"/>
   </visual>
   <collision>
-    <origin xyz="0.0 -0.181075 0.0556" rpy="1.5708 0 0"/>
+    <origin xyz="0.0 -0.4 0.0" rpy="0 0 0"/>
     <geometry>
-      <cylinder radius="0.05" length="0.02"/>
+      <mesh filename="package://fcl_coll/meshes/left_wheel_1.stl" scale="0.001 0.001 0.001"/>
     </geometry>
   </collision>
@@ -81,5 +81,5 @@
     <origin xyz="-0.0 -0.0 -0.0" rpy="0 0 0"/>
     <geometry>
-      <cylinder radius="0.05" length="0.02"/>
+      <mesh filename="package://fcl_coll/meshes/imu_1.stl" scale="0.001 0.001 0.001"/>
     </geometry>
     <material name="silver"/>
@@ -88,5 +88,5 @@
     <origin xyz="-0.0 -0.0 -0.0" rpy="0 0 0"/>
     <geometry>
-      <cylinder radius="0.05" length="0.02"/>
+      <mesh filename="package://fcl_coll/meshes/imu_1.stl" scale="0.001 0.001 0.001"/>
     </geometry>
   </collision>
@@ -101,5 +101,5 @@
     <origin xyz="-0.087 -0.0 -0.0065" rpy="0 0 0"/>
     <geometry>
-      <cylinder radius="0.05" length="0.02"/>
+      <mesh filename="package://fcl_coll/meshes/gps_1.stl" scale="0.001 0.001 0.001"/>
     </geometry>
     <material name="silver"/>
@@ -108,5 +108,5 @@
     <origin xyz="-0.087 -0.0 -0.0065" rpy="0 0 0"/>
     <geometry>
-      <cylinder radius="0.05" length="0.02"/>
+      <mesh filename="package://fcl_coll/meshes/gps_1.stl" scale="0.001 0.001 0.001"/>
     </geometry>
   </collision>
@@ -121,5 +121,5 @@
     <origin xyz="-0.2625 -0.0 -0.0085" rpy="0 0 0"/>
     <geometry>
-      <cylinder radius="0.05" length="0.02"/>
+      <mesh filename="package://fcl_coll/meshes/Lidar_1.stl" scale="0.001 0.001 0.001"/>
     </geometry>
     <material name="silver"/>
@@ -128,5 +128,5 @@
     <origin xyz="-0.2625 -0.0 -0.0085" rpy="0 0 0"/>
     <geometry>
-     <cylinder radius="0.05" length="0.02"/>
+      <mesh filename="package://fcl_coll/meshes/Lidar_1.stl" scale="0.001 0.001 0.001"/>
     </geometry>
   </collision>
@@ -139,8 +139,8 @@
 </joint>
 <joint name="left_motor_joint" type="continuous">
-  <origin xyz="0.0 0.181075 -0.0556" rpy="0 0 0"/>
+  <origin xyz="0.0 -0.4 0.0" rpy="0 0.0 0"/>
   <parent link="base_link"/>
   <child link="left_wheel_1"/>
-  <axis xyz="-0.0 1.0 0.0"/>
+  <axis xyz="-0.0 -0.4 0.0"/>
 </joint>
 <joint name="Rigid 15" type="fixed">
