Commit message: minnor changes

File: PXA-100_description/urdf/px.urdf (robot description, URDF)
Before this commit: robot PXA-100, 8 links, 7 joints
Links:
- link end: geometry collision box size=0.0 0.0 0.0; visual box size=0.01 0.01 0.01
Joints:
- joint Revolute 15: limit (none) -> lower=-1000 upper=1000 effort=5 velocity=1.0
- joint Revolute 18: limit (none) -> lower=-1000 upper=1000 effort=5 velocity=1.0
- joint Revolute 19: limit (none) -> lower=-1000 upper=1000 effort=5 velocity=1.0
- joint Revolute 20: limit (none) -> lower=-1000 upper=1000 effort=5 velocity=1.0
- joint box_joint: limit (none) -> lower=-1000 upper=1000 effort=5 velocity=1.0
